File: 8inch-adapter-pcb/fd50to34.kicad_pcb (KiCad board)
At the start: 2 copper layers, 27.9 x 68.6 mm, 2 parts, among them J1 61205022121, J2 61203422121

Commit message: rev2 pcb
Parts:
- added J3: TWO_SIDES, Connector_PinHeader_2.54mm:PinHeader_1x02_P2.54mm_Vertical, F.Cu at (10.2, 10.2)
Connections:
- J1 pad 10: GND -> Net-(J1-~{FD2S})
Routing:
- net Net-(J1-~{FD2S}): track 0.00 -> 5.08 mm
