File: 8inch-adapter-pcb/fd50to34.kicad_sch (KiCad schematic)
At the start: 2 parts, among them J1 61205022121, J2 61203422121

Commit message: rev2 pcb
Parts:
- added J3: TWO_SIDES, Connector_PinHeader_2.54mm:PinHeader_1x02_P2.54mm_Vertical, symbol Connector:Conn_01x02_Pin
Connections:
- net GND: now also J3.1 (Pin_1); no longer J1.10 (~{FD2S})
- new net: J1.10 (~{FD2S}), J3.2 (Pin_2)
Changed lines of the file:
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@@
   (junction (at 44.45 71.12) (diameter 0) (color 0 0 0 0)
-  )
-  (junction (at 46.99 73.66) (diameter 0) (color 0 0 0 0)
   )
   (junction (at 44.45 81.28) (diameter 0) (color 0 0 0 0)
@@
     (stroke (width 0) (type default))
   )
-  (wire (pts (xy 46.99 73.66) (xy 82.55 73.66))
-    (stroke (width 0) (type default))
-  )
   (wire (pts (xy 46.99 86.36) (xy 44.45 86.36))
     (stroke (width 0) (type default))
@@
     (stroke (width 0) (type default))
   )
+  (wire (pts (xy 95.885 73.66) (xy 91.44 73.66))
+    (stroke (width 0) (type default))
+  )
   (wire (pts (xy 196.85 76.2) (xy 196.85 83.82))
     (stroke (width 0) (type default))
@@
     (stroke (width 0) (type default))
   )
+  (wire (pts (xy 88.9 73.66) (xy 88.9 71.755))
+    (stroke (width 0) (type default))
+  )
   (wire (pts (xy 232.41 88.9) (xy 236.22 88.9))
     (stroke (width 0) (type default))
@@
     (stroke (width 0) (type default))
   )
+  (wire (pts (xy 91.44 73.66) (xy 91.44 71.755))
+    (stroke (width 0) (type default))
+  )
   (wire (pts (xy 46.99 73.66) (xy 44.45 73.66))
     (stroke (width 0) (type default))
@@
   )
   (wire (pts (xy 44.45 78.74) (xy 44.45 76.2))
+    (stroke (width 0) (type default))
+  )
+  (wire (pts (xy 82.55 73.66) (xy 88.9 73.66))
     (stroke (width 0) (type default))
   )
@@
         )
       )
+    )
+  )
+  (symbol (lib_id "Connector:Conn_01x02_Pin") (at 91.44 66.675 270) (unit 1)
+    (in_bom yes) (on_board yes) (dnp no) (fields_autoplaced)
+    (property "Reference" "J3" (at 92.71 66.04 90)
+      (effects (font (size 1.27 1.27)) (justify left))
+    )
+    (property "Value" "TWO_SIDES" (at 92.71 68.58 90)
+      (effects (font (size 1.27 1.27)) (justify left))
+    )
+    (property "Footprint" "Connector_PinHeader_2.54mm:PinHeader_1x02_P2.54mm_Vertical" (at 91.44 66.675 0)
+      (effects (font (size 1.27 1.27)) hide)
+    )
+    (property "Datasheet" "~" (at 91.44 66.675 0)
+      (effects (font (size 1.27 1.27)) hide)
+    )
+    (pin "1")
+    (pin "2")
+    (instances
+      (project "fd50to34"
+        (path "/3358d231-6770-4f6a-b19f-5f44807fda78"
+          (reference "J3") (unit 1)
+        )
+      )
+    )
+  )
+  (symbol (lib_id "fd50to34-rescue:GND") (at 95.885 73.66 90) (unit 1)
+    (in_bom yes) (on_board yes) (dnp no)
+    (property "Reference" "#PWR03" (at 102.235 73.66 0)
+      (effects (font (size 1.524 1.524)) hide)
+    )
+    (property "Value" "GND" (at 99.695 73.66 0)
+      (effects (font (size 1.524 1.524)))
+    )
+    (property "Footprint" "" (at 95.885 73.66 0)
+      (effects (font (size 1.524 1.524)))
+    )
+    (property "Datasheet" "" (at 95.885 73.66 0)
+      (effects (font (size 1.524 1.524)))
+    )
+    (pin "1")
+    (instances
+      (project "fd50to34"
+        (path "/3358d231-6770-4f6a-b19f-5f44807fda78"
+          (reference "#PWR03") (unit 1)
+        )
+      )
